File: KiCad/hackpad.kicad_pcb (KiCad board)
At the start: 2 copper layers, 92.3 x 64.8 mm, 11 parts, among them SW1 RotaryEncoder_Switch, SW2 RotaryEncoder_Switch, SW3 RotaryEncoder_Switch, SW4 SW_Push, SW5 SW_Push, SW6 SW_Push, U1 Seeed Studio XIAO SAMD21, U2 PCF8574A

Commit message: PCB V3.5 KiCad Files Update
Parts:
- OL1: footprint kbd:OLED -> KiCad-SSD1306-0.91-OLED-4pin-128x32.pretty-master:SSD1306-0.91-OLED-4pin-128x32
- moved OL1 39.4 mm to (195.0, 99.8), turned to 180 degrees
- moved G*** 1.36 mm to (201.5, 92.5)
Routing:
- net GND: track 353.3 -> 350.0 mm
- net VCC: track 72.1 -> 75.3 mm
- net Net-(OL1-SDA): track 71.7 -> 73.6 mm
- net Net-(OL1-SCL): track 72.4 -> 73.4 mm, vias 1 -> 3
Other:
- outline, holes or cut-outs redrawn
- board text added: "10/14/24"
- board text added: "5V"
- board text added: "D0"
- board text added: "D1"
- board text added: "D10"
- board text added: "D2"
- board text added: "D3"
- board text added: "D7"
- board text added: "D8"
- board text added: "D9"
- board text added: "EC11"
- board text added: "GND"
- board text added: "HackPad V3.5"
- board text added: "I messed up (again)"
- board text added: "IO_INT"
- board text added: "OLED (128x32)"
- board text added: "P0"
- board text added: "P1"
- board text added: "P2"
- board text added: "P3"
- board text added: "P4"
- board text added: "P5"
- board text added: "P6"
- board text added: "P7"
- board text added: "SCL"
- board text added: "SDA"
- board text added: "VCC"
