File: KiCad/hackpad.kicad_sch (KiCad schematic)
At the start: 10 parts, among them SW1 RotaryEncoder_Switch, SW2 RotaryEncoder_Switch, SW3 RotaryEncoder_Switch, SW4 SW_Push, SW5 SW_Push, SW6 SW_Push, U1 Seeed Studio XIAO SAMD21, U2 PCF8574A

Commit message: PCB V3.5 KiCad Files Update
Parts:
- OL1: footprint kbd:OLED -> KiCad-SSD1306-0.91-OLED-4pin-128x32.pretty-master:SSD1306-0.91-OLED-4pin-128x32
Changed lines of the file:
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@@
 			)
 		)
-		(property "Footprint" "kbd:OLED"
+		(property "Footprint" "KiCad-SSD1306-0.91-OLED-4pin-128x32.pretty-master:SSD1306-0.91-OLED-4pin-128x32"
 			(at 201.93 39.37 0)
 			(effects
